File: Курс 3/Архитектура ЭВМ/Курисовая/2BKeyboard/2BKeyboard.kicad_pcb (KiCad board)
At the start: 2 copper layers, 4 parts

Commit message: vault backup: 2026-03-25 01:54:36
Routing:
- net (no net): track 300.7 -> 410.7 mm
Changed lines of the file:
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@@
+	)
+	(segment
+		(start 48.5 24)
+		(end 48.5 38)
+		(width 0.25)
+		(layer "F.Cu")
+		(net "")
 	)
 	(segment
@@
 	)
 	(segment
+		(start 54.5 44)
+		(end 54.62 44)
+		(width 0.25)
+		(layer "F.Cu")
+		(net "")
+	)
+	(segment
+		(start 48.5 38)
+		(end 54.5 44)
+		(width 0.25)
+		(layer "F.Cu")
+		(net "")
+	)
+	(segment
+		(start 99.74 57.68)
+		(end 99.74 49.24)
+		(width 0.25)
+		(layer "F.Cu")
+		(net "")
+	)
+	(segment
+		(start 99.74 49.24)
+		(end 77.5 27)
+		(width 0.25)
+		(layer "F.Cu")
+		(net "")
+	)
+	(segment
 		(start 51.74 58.8)
 		(end 51.74 77.18)
@@
 	)
 	(segment
+		(start 77.5 23.5)
+		(end 74 20)
+		(width 0.25)
+		(layer "F.Cu")
+		(net "")
+	)
+	(segment
 		(start 92.12 57.68)
 		(end 92.12 51.06)
@@
 	)
 	(segment
-		(start 91.4 42.34)
-		(end 70.74 42.34)
-		(width 0.25)
-		(layer "F.Cu")
-		(net "")
-	)
-	(segment
-		(start 97.24 51.18)
-		(end 97.2 51.22)
-		(width 0.25)
-		(layer "F.Cu")
-		(net "")
-	)
-	(segment
-		(start 99.74 57.68)
-		(end 99.74 50.68)
-		(width 0.25)
-		(layer "F.Cu")
-		(net "")
-	)
-	(segment
-		(start 49.24 37.18)
-		(end 49.32 37.26)
+		(start 52.5 20)
+		(end 48.5 24)
 		(width 0.25)
 		(layer "F.Cu")
@@
 	)
 	(segment
+		(start 77.5 27)
+		(end 77.5 23.5)
+		(width 0.25)
+		(layer "F.Cu")
+		(net "")
+	)
+	(segment
 		(start 94.74 51.18)
 		(end 83.36 39.8)
@@
 	)
 	(segment
+		(start 55.5 39.8)
+		(end 46.62 39.8)
+		(width 0.25)
+		(layer "F.Cu")
+		(net "")
+	)
+	(segment
+		(start 51 25.5)
+		(end 54 22.5)
+		(width 0.25)
+		(layer "F.Cu")
+		(net "")
+	)
+	(segment
 		(start 51.74 77.18)
 		(end 61.86 77.18)
@@
 	)
 	(segment
+		(start 51 37.84)
+		(end 51 25.5)
+		(width 0.25)
+		(layer "F.Cu")
+		(net "")
+	)
+	(segment
 		(start 47.78 58.14)
 		(end 53.42 52.5)
@@
 	)
 	(segment
-		(start 99.74 50.68)
-		(end 91.4 42.34)
-		(width 0.25)
-		(layer "F.Cu")
-		(net "")
-	)
-	(segment
 		(start 41.43 44.99)
-		(end 49.24 37.18)
+		(end 46.62 39.8)
+		(width 0.25)
+		(layer "F.Cu")
+		(net "")
+	)
+	(segment
+		(start 97.2 50.2)
+		(end 97.2 57.68)
 		(width 0.25)
 		(layer "F.Cu")
@@
 	)
 	(segment
-		(start 70.74 44.88)
-		(end 90.94 44.88)
-		(width 0.25)
-		(layer "F.Cu")
-		(net "")
-	)
-	(segment
 		(start 55.5 55.04)
 		(end 51.74 58.8)
@@
 	)
 	(segment
-		(start 97.2 51.22)
-		(end 97.2 57.68)
+		(start 74 20)
+		(end 52.5 20)
+		(width 0.25)
+		(layer "F.Cu")
+		(net "")
+	)
+	(segment
+		(start 75 25)
+		(end 75 28)
+		(width 0.25)
+		(layer "F.Cu")
+		(net "")
+	)
+	(segment
+		(start 54.62 44)
+		(end 55.5 44.88)
+		(width 0.25)
+		(layer "F.Cu")
+		(net "")
+	)
+	(segment
+		(start 75 28)
+		(end 97.2 50.2)
+		(width 0.25)
+		(layer "F.Cu")
+		(net "")
+	)
+	(segment
+		(start 55.5 42.34)
+		(end 51 37.84)
+		(width 0.25)
+		(layer "F.Cu")
+		(net "")
+	)
+	(segment
+		(start 54 22.5)
+		(end 72.5 22.5)
 		(width 0.25)
 		(layer "F.Cu")
@@
 	)
 	(segment
-		(start 49.32 37.26)
-		(end 55.5 37.26)
+		(start 72.5 22.5)
+		(end 75 25)
 		(width 0.25)
 		(layer "F.Cu")
@@
 		(width 0.25)
 		(layer "F.Cu")
-		(net "")
-	)
-	(segment
-		(start 90.94 44.88)
-		(end 97.24 51.18)
-		(width 0.25)
-		(layer "F.Cu")
